File: pcb/FPGA_MSXtR_Stack_SLOT/StackSlot.kicad_sch (KiCad schematic)
At the start: 30 parts, among them J1 Conn_01x01, J2 Conn_01x01, J5 MSX_EXBUS_B, J6 MSX_EXBUS_A

Commit message: Bugfix Pico Firmware
Other:
- note added: "SLOT_DATA_DIR 1: CPU → Cartridge (WRITE) 0: CPU ← Cartridge (READ)"
- note removed: "BUSDIR 0: CPU → Cartridge (WRITE) 1: CPU ← Cartridge (READ)"
Changed lines of the file:
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@@
 		)
 	)
-	(text "BUSDIR\n0: CPU → Cartridge (WRITE)\n1: CPU ← Cartridge (READ)"
+	(text "SLOT_DATA_DIR\n1: CPU → Cartridge (WRITE)\n0: CPU ← Cartridge (READ)"
 		(exclude_from_sim no)
 		(at 247.396 31.496 0)
