File: pcb/FPGA_MSXtR_Stack_CPU2/StackCPU.kicad_sch (KiCad schematic)
At the start: 48 parts, among them J1 MSX_EXBUS_A, J2 MSX_EXBUS_B, J3 Conn_02x06_Odd_Even, J4 Micro_SD_Card, J5 Keybard I2C Connector, J6 USB_C_Receptacle_PowerOnly_6P, SW1 SW_MEC_5G, SW2 SW_SPDT, SW3 SW_DIP_x04, U10 W25Q32JVSS

Commit message: Updated PCB
Parts:
- removed C9: 0.1uF, Capacitor_SMD:C_0402_1005Metric, symbol Device:C
- removed J3: Conn_02x06_Odd_Even, Connector_PinSocket_2.54mm:PinSocket_2x06_P2.54mm_Vertical, symbol Connector_Generic:Conn_02x06_Odd_Even
- removed U10: W25Q32JVSS, Package_SO:SOIC-8_5.3x5.3mm_P1.27mm, symbol Memory_Flash:W25Q32JVSS
- added R17, R18, R23, R24, R25, R26, R27, R28: 3.3K, Resistor_SMD:R_0402_1005Metric, symbol Device:R
- U1: symbol My Parts:FPGA_MSX_CPU(UPPER) -> My Parts:FPGA_MSXtR_CPU2(UPPER)
- U2: symbol My Parts:FPGA_MSX_CPU(LOWER) -> My Parts:FPGA_MSXtR_CPU2(LOWER)
Connections:
- net JTAG_TCK is gone; now on net +3V3: U1.21 (HS_SIO3)
- net JTAG_TDI is gone; now on net HS_CLK: U1.27 (HS_SIO0)
- net JTAG_TDO is gone; now on net GND: U1.25 (HS_SIO1)
- net SLOT_SLTSL0_N is gone; now on net SLOT_A0: J1.4 (Pin_4)
- net SLOT_SLTSL3_N is gone; now on net SLOT_A2: J1.6 (Pin_6)
- net SMEM_SCLK is gone; now on net SRAM_SCLK: R8.2, U1.7 (SRAM_SCLK)
- net SMEM_SIO0 is gone; now on net SRAM_SIO0: R9.2, U1.9 (SRAM_SIO0)
- net SMEM_SIO1 is gone; now on net SRAM_SIO1: R10.2, U1.11 (SRAM_SIO1)
- net SMEM_SIO3 is gone; now on net HS_CLK: R12.1, U1.17 (HS_CLK)
- net SROM_MOSI is gone; now on net SLOT_ROM1_CE_N: R21.1, U2.116 (SLOT_ROM1_CE_N)
- net +12V: now also J1.37 (Pin_37); no longer J1.38 (Pin_38)
- net +3V3: now also J1.34 (Pin_34), J2.39 (Pin_39), R11.1, R17.1, R17.2, R18.2, R23.2, R24.2, R25.1, R26.2, R27.1, R28.1; no longer J2.35 (Pin_35), J5.3 (Pin_3), R11.2
- net +5V: now also J1.35 (Pin_35), J5.3 (Pin_3); no longer J1.34 (Pin_34), J2.39 (Pin_39)
- net -12V: now also J1.39 (Pin_39); no longer J1.40 (Pin_40)
- net GND: now also J1.19 (Pin_19), J1.20 (Pin_20), J1.21 (Pin_21), J1.23 (Pin_23), J1.24 (Pin_24), J1.25 (Pin_25), J1.27 (Pin_27), J1.28 (Pin_28), J1.38 (Pin_38), R23.1; no longer J1.36 (Pin_36), J2.37 (Pin_37)
- net I2C_SCL: now also J5.1 (Pin_1), R28.2; no longer J5.2 (Pin_2)
- net I2C_SDA: now also J5.2 (Pin_2), R27.2; no longer J5.1 (Pin_1)
- net MCU_CS_N: now also R19.1, U1.28 (MCU_CS_N); no longer U1.14 (MCU_CS_N)
- net MCU_INTR: now also U1.36 (MCU_INTR); no longer U2.83 (MCU_INTR)
- net MCU_MISO: now also J2.35 (Pin_35), R16.1, U1.32 (MCU_MISO); no longer U1.20 (MCU_MISO)
- net MCU_MOSI: now also J2.37 (Pin_37), R15.1, U1.30 (MCU_MOSI); no longer U1.18 (MCU_MOSI)
- net MCU_SCLK: now also J2.31 (Pin_31), U1.34 (MCU_SCLK), R26.1; no longer U1.16 (MCU_SCLK)
- net SLOT_A0: now also U2.93 (SLOT_A0); no longer J1.25 (Pin_25), U2.63 (SLOT_A0)
- net SLOT_A1: now also J1.1 (Pin_1), U2.95 (SLOT_A1); no longer J2.26 (Pin_26), U2.65 (SLOT_A1)
- net SLOT_A10: now also J2.20 (Pin_20), U2.68 (SLOT_A10); no longer J1.17 (Pin_17), U2.78 (SLOT_A10)
- net SLOT_A11: now also J2.19 (Pin_19), U2.66 (SLOT_A11); no longer J2.18 (Pin_18), U2.76 (SLOT_A11)
- net SLOT_A12: now also J2.23 (Pin_23); no longer J2.22 (Pin_22)
- net SLOT_A13: now also J1.2 (Pin_2), U2.80 (SLOT_A13); no longer J1.23 (Pin_23), U11.4 (A13), U12.4 (A13), U2.72 (SLOT_A13)
- net SLOT_A14: now also J2.25 (Pin_25), U2.78 (SLOT_A14); no longer J2.24 (Pin_24), U11.5 (A14), U12.5 (A14), U2.108 (SLOT_A14)
- net SLOT_A15: now also J2.18 (Pin_18), U2.83 (SLOT_A15); no longer J1.15 (Pin_15), U11.11 (A15), U12.11 (A15), U2.106 (SLOT_A15)
- net SLOT_A2: now also U2.97 (SLOT_A2); no longer J1.27 (Pin_27), U2.67 (SLOT_A2)
- net SLOT_A3: now also J1.3 (Pin_3), U2.99 (SLOT_A3); no longer J2.28 (Pin_28), U2.69 (SLOT_A3)
- net SLOT_A4: now also J1.8 (Pin_8), U2.101 (SLOT_A4); no longer J1.29 (Pin_29), U2.71 (SLOT_A4)
- net SLOT_A5: now also J1.5 (Pin_5), U2.103 (SLOT_A5); no longer J2.30 (Pin_30), U2.73 (SLOT_A5)
- net SLOT_A6: now also J2.22 (Pin_22), U2.72 (SLOT_A6); no longer J1.19 (Pin_19), U2.93 (SLOT_A6)
- net SLOT_A7: now also J2.21 (Pin_21), U2.70 (SLOT_A7); no longer J2.20 (Pin_20), U2.95 (SLOT_A7)
- net SLOT_A8: now also J2.24 (Pin_24), U2.76 (SLOT_A8); no longer J1.21 (Pin_21), U2.82 (SLOT_A8)
- net SLOT_A9: now also J2.17 (Pin_17), U2.73 (SLOT_A9); no longer J2.16 (Pin_16), U2.80 (SLOT_A9)
- net SLOT_CLOCK_N: now also J1.18 (Pin_18), U2.90 (SLOT_CLOCK_N); no longer J1.39 (Pin_39), U2.77 (SLOT_CLOCK_N(READY))
- net SLOT_CS12_N: now also J2.3 (Pin_3), U1.10 (SLOT_CS12_N); no longer J2.4 (Pin_4), U2.85 (SLOT_CS12_N(DONE))
- net SLOT_CS1_N: now also J2.1 (Pin_1), U1.6 (SLOT_CS1_N); no longer J2.2 (Pin_2), U1.10 (SLOT_CS1_N)
- net SLOT_CS2_N: now also J2.2 (Pin_2), U1.8 (SLOT_CS2_N); no longer J1.1 (Pin_1), U1.12 (SLOT_CS2_N)
- net SLOT_D0: now also J1.10 (Pin_10), U2.94 (SLOT_D0); no longer J1.31 (Pin_31), U2.90 (SLOT_D0)
- net SLOT_D1: now also J1.7 (Pin_7), U2.96 (SLOT_D1); no longer J2.32 (Pin_32), U2.92 (SLOT_D1)
- net SLOT_D2: now also J1.12 (Pin_12), U2.98 (SLOT_D2); no longer J1.33 (Pin_33), U2.94 (SLOT_D2)
- net SLOT_D3: now also J1.9 (Pin_9), U2.100 (SLOT_D3); no longer J2.34 (Pin_34), U2.96 (SLOT_D3)
- net SLOT_D4: now also J1.14 (Pin_14), U2.102 (SLOT_D4); no longer J1.35 (Pin_35), U2.98 (SLOT_D4)
- net SLOT_D5: now also J1.11 (Pin_11), U2.104 (SLOT_D5); no longer J2.36 (Pin_36), U2.100 (SLOT_D5)
- net SLOT_D6: now also J1.16 (Pin_16), U2.106 (SLOT_D6); no longer J1.37 (Pin_37), U2.102 (SLOT_D6)
- net SLOT_D7: now also J1.13 (Pin_13), U2.108 (SLOT_D7); no longer J2.38 (Pin_38), U2.104 (SLOT_D7)
- net SLOT_DATA_DIR: now also J2.26 (Pin_26), U2.82 (SLOT_DATA_DIR); no longer J2.5 (Pin_5), U1.6 (SLOT_DATA_DIR)
- net SLOT_INT_N: now also J2.8 (Pin_8), U1.20 (SLOT_INT_N); no longer J1.7 (Pin_7), U2.97 (SLOT_INT_N)
- net SLOT_IORQ_N: now also J2.11 (Pin_11), U1.26 (SLOT_IORQ_N); no longer J2.10 (Pin_10), U2.68 (SLOT_IORQ_N)
- net SLOT_M1_N: now also J2.9 (Pin_9), U1.22 (SLOT_M1_N); no longer J2.8 (Pin_8), U1.3 (SLOT_M1_N)
- net SLOT_MERQ_N: now also J2.12 (Pin_12), U2.63 (SLOT_MERQ_N); no longer J1.11 (Pin_11), U2.70 (SLOT_MERQ_N)
- net SLOT_OE_N: now also J2.16 (Pin_16), U2.71 (SLOT_OE_N); no longer J2.7 (Pin_7), R7.2, U1.5 (SLOT_OE_N)
- net SLOT_RD_N: now also J2.14 (Pin_14), U2.67 (SLOT_RD_N); no longer J1.13 (Pin_13), U2.109 (SLOT_RD_N)
- net SLOT_RESET_N: now also J2.15 (Pin_15), U2.69 (SLOT_RESET_N); no longer J2.14 (Pin_14), U2.101 (SLOT_RESET_N)
- net SLOT_RFSH_N: now also J2.6 (Pin_6), U1.16 (SLOT_RFSH_N); no longer J1.2 (Pin_2), U2.66 (SLOT_RFSH_N)
- net SLOT_ROM0_CE_N: now also R20.1, U2.114 (SLOT_ROM0_CE_N); no longer U1.8 (SLOT_ROM0_CE_N)
- net SLOT_ROM1_CE_N: no longer U2.117 (SLOT_ROM1_CE_N)
- net SLOT_SLTSL1_N: now also J2.4 (Pin_4), U1.12 (SLOT_SLTSL1_N); no longer J1.3 (Pin_3), U1.26 (SRAM_CS2_N)
- net SLOT_SLTSL2_N: now also J2.5 (Pin_5), U1.14 (SLOT_SLTSL2_N); no longer J1.5 (Pin_5), U1.28 (SRAM_CS3_N)
- net SLOT_WAIT_N: now also J2.7 (Pin_7), U1.18 (SLOT_WAIT_N); no longer J2.6 (Pin_6), U2.99 (SLOT_WAIT_N)
- net SLOT_WR_N: now also J2.13 (Pin_13); no longer J2.12 (Pin_12), U2.107 (SLOT_WR_N)
- net SRAM_CS_N: now also R7.2, U1.5 (SRAM_CS_N); no longer R15.1, U1.22 (SRAM_CS0_N)
- net SRAM_SIO2: now also R11.2, U1.15 (SRAM_SIO2)
- net SRAM_SIO3: now also U1.3 (SRAM_SIO3), R25.2
- net OSD_SPI_CS_N: now reaches U4.4 (FPGA_OSD_SPI_CS_N(GP2))
- net OSD_SPI_CS_N: now also J2.33 (Pin_33)
- net HS_READY: now reaches J1.30 (Pin_30)
- net HS_CLK: now reaches J1.32 (Pin_32)
- net HS_CLK: now also J1.40 (Pin_40), R24.1
- net JTAG_TMS renamed HS_SIO2
- net HS_SIO2: now also J1.36 (Pin_36), R18.1
- net SLOT_A16 renamed SLOT_MA16
- net SLOT_MA16: now also U2.113 (SLOT_MA16); no longer U2.111 (SLOT_A16)
- net SLOT_A17 renamed SLOT_MA17
- net SLOT_MA17: now also U2.115 (SLOT_MA17); no longer U2.113 (SLOT_A17)
- net SLOT_A18 renamed SLOT_MA18
- net SLOT_MA18: now also U2.117 (SLOT_MA18); no longer U2.115 (SLOT_A18)
- removed net SLOT_BUSDIR_N: J1.9 (Pin_9), U2.103 (SLOT_BUSDIR_N)
- removed net SMEM_SIO2: R11.1, U1.15 (SRAM_SIO2)
- net SROM_CS_N renamed SLOT_BUSDIR
- net SLOT_BUSDIR: now also J2.10 (Pin_10); no longer R16.1
- net SROM_MISO renamed HS_CS_N
- net HS_CS_N: now also J1.33 (Pin_33)
- net SROM_SCLK: no longer names the net of U2.112 (未使用)
- net SROM_SCLK: no longer R19.1
- net UART_RX: no longer names the net of U2.79 (UART_RX)
- net UART_TX: no longer names the net of U2.81 (UART_TX)
- new net SLOT_MA13: U11.4 (A13), U12.4 (A13), U2.107 (SLOT_MA13)
- new net SLOT_MA14: U11.5 (A14), U12.5 (A14), U2.109 (SLOT_MA14)
- new net SLOT_MA15: U11.11 (A15), U12.11 (A15), U2.111 (SLOT_MA15)
- new net WR_N: U2.65 (SLOT_WR_N)
- no-connect marks 56 -> 41
Other:
- note added: "LCSC Part#C43651917 Flash ROM 4Mbit Extend ROM (OPTION) SST39VF040-70"
- note added: "MSX_EXBUS_B"
- note added: "MSXtR PICO"
- note added: "SLOT_SNDIN1"
- note added: "SLOT_SNDIN2"
- note removed: "3V3"
- note removed: "5V"
- note removed: "FPGAサイドの TXO/RXO を、 コネクタの RX/TX にクロスで接続する。"
- note removed: "GND"
- note removed: "LCSC Part#C43651917 Flash ROM 4Mbit Extend ROM SST39VF040-70"
- note removed: "LCSC Part#C82344 Kanji ROM"
- note removed: "RTS"
- note removed: "RX"
- note removed: "SLOT_SNDIN"
- note removed: "TCK"
- note removed: "TDI"
- note removed: "TDO"
- note removed: "TDR"
- note removed: "TMS"
- note removed: "TX"
- note removed: "TangPrimer20K Lite に付属する UARTモジュールのピンアサイン"
- moved on the sheet: C10, C11, C7, J1, J2, J5, R10, R15, R16, R20, R21, R22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
